File: eagle/miner.sch (EAGLE design)
At the start: 30 parts, among them IC1 A3255-Q48

Commit message: miner with PIC
Parts:
- removed CONFIG_NI, CONFIG_PI, REPORT_N, REPORT_P, RSTN, XCLKIN: LSP10, solpad:LSP10
- added AVALON1: A3255-Q48, avalon:A3255-Q48
- added C14: 22p, rcl:C-EUC0805
- added C15, C16, C17, C18, C19: 100n, rcl:C-EUC0805
- added IC2: 74LS14, 74xx-eu:74LS14D
- added IC3: 74LVC1G14SE-7, 74xx-little-de:74AHC1G32DCK
- added IC4, U$1: TCN75, miner:TCN75
- added JP1: PICkit 3, pinhead:PINHD-1X6
- added Q1: SI501, miner:SI501
- added R10, R11, R12, R13, R14, R15, R16, R17, R19, R20, R6, R7, R8, R9: 33, rcl:R-EU_R0805
- added R18: 3k3, rcl:R-EU_R0805
- added R5: 1k, rcl:R-EU_R0805
- added U1RX, U1TX: LSP10, solpad:LSP10
- IC1: value A3255-Q48 -> PIC32MX220F032B; device avalon:A3255-Q48 -> miner:PIC32MX220F032B
- R4: value 33 -> 3k3
Connections:
- new net CLK1: AVALON1.XCLKIN, R8.1
- new net CLK10: R17.1
- new net CLK2: R9.1
- new net CLK3: R10.1
- new net CLK4: R11.1
- new net CLK5: R12.1
- new net CLK6: R13.1
- new net CLK7: R14.1
- new net CLK8: R15.1
- new net CLK9: R16.1
- new net N$11: Q1.OUT, R6.2, R7.2
- new net N$12: IC2A.I, R7.1
- new net N$13: IC2D.O, R5.1
- new net N$14: C14.1, IC2E.I, R5.2
- new net N$15: IC2A.O, IC2B.I, IC2C.I
- new net N$16: IC2B.O, R10.2, R11.2, R12.2, R8.2, R9.2
- new net N$17: IC2C.O, R13.2, R14.2, R15.2, R16.2, R17.2
- new net N$18: IC1.OSC1/CLKI/RPA2/RA2, R6.1
- new net N$19: IC1.!MCLR, JP1.1
- new net N$20: R19.1, U1TX.MP
- new net N$21: IC1.PGED3/VREF+/CVREF+/AN0/C3INC/RPA0/CTED1/PMD7/RA0, JP1.4
- new net N$22: IC1.PGEC3/VREF-/CVREF-/AN1/RPA1/CTED2/PMD6/RA1, JP1.5
- new net N$23: R20.1, U1RX.MP
- new net OR: IC2D.I, IC3A.O
- new net OR_DELAY: IC1.AN9/C3INA/RPB15/SCK2/CTED6/PMCS1/RB15, IC2E.O
- new net REPORT_N: AVALON1.REPORT_N, AVALON1.REPORT_P, IC2F.I, IC3A.I0, R2.1, R3.1
- new net REPORT_N_I: IC1.AN4/C1INB/C2IND/RPB2/SDA2/CTED13/PMD2/RB2, IC2F.O
- new net REPORT_P: IC3A.I1
- net +3V3: now also AVALON1.OVDD, C15.1, C16.1, C17.1, C18.1, C19.1, IC1.AVDD, IC1.VDD, IC2P.VCC, IC3P.VCC, IC4.VDD, JP1.2, Q1.VDD, R18.1, R4.1; no longer IC1.OVDD
- net GND: now also AVALON1.GND, C14.2, C15.2, C16.2, C17.2, C18.2, C19.2, IC1.AVSS, IC1.VSS, IC2P.GND, IC3P.GND, IC4.A0, IC4.A1, IC4.A2, IC4.GND, JP1.3, Q1.GND; no longer IC1.GND
- net N$1: now also AVALON1.RSTN, IC1.OSC2/CLKO/RPA3/PMA0/RA3; no longer IC1.RSTN, RSTN.MP
- net N$10: now also AVALON1.CORE_CLKOUT; no longer IC1.CORE_CLKOUT
- net N$2: now also IC1.TDO/RPB9/SDA1/CTED4/PMD3/RB9, IC4.SDA, R4.2; no longer IC1.REPORT_N, R2.1, REPORT_N.MP
- net N$3: now also IC1.TCK/RPB8/SCL1/CTED10/PMD4/RB8, IC4.SCL, R18.2; no longer IC1.REPORT_P, R3.1, REPORT_P.MP
- net N$4: now also IC1.SOSCI/RPB4/RB4, R19.2; no longer IC1.XCLKIN, R4.2
- net N$5: now also IC1.AN11/RPB13/CTPLS/PMRD/RB13, R20.2; no longer R4.1, XCLKIN.MP
- net N$6: now also AVALON1.CONFIG_PI, IC1.SOSCO/RPA4/T1CK/CTED9/PMA1/RA4; no longer CONFIG_PI.MP, IC1.CONFIG_PI
- net N$7: now also AVALON1.CONFIG_NI, IC1.PGED1/AN2/C1IND/C2INB/C3IND/RPB0/PMD0/RB0; no longer CONFIG_NI.MP, IC1.CONFIG_NI
- net N$8: now also AVALON1.CONFIG_PO; no longer IC1.CONFIG_PO
- net N$9: now also AVALON1.CONFIG_NO; no longer IC1.CONFIG_NO
- net VDD: now also AVALON1.DVDD, AVALON1.VDDA_PLL, AVALON1.VDD_PLL; no longer IC1.DVDD, IC1.VDDA_PLL, IC1.VDD_PLL
Other:
- moved on the sheet: 0.9V, 3V3, C1, C10, C11, C12, C13, C2, C3, C4, C5, C6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

Commit message: FPGA implementation converted to PIC firmware
Parts:
- removed U$1: TCN75, miner:TCN75
- added C20: 10u, rcl:C-EUC0805
- added CLK-OUT: LSP10, solpad:LSP10
- added LED1: (no value), led:LED5MM
- added R21: 10k, rcl:R-EU_R0805
- added R22: 1k, rcl:R-EU_R0805
- IC2: value 74LS14 -> 74LCX14
Connections:
- net N$19 renamed VPP
- net N$21 renamed PGD
- net N$22 renamed PGC
- new net N$19: C20.1, IC1.VCAP
- new net N$21: CLK-OUT.MP, IC1.OSC2/CLKO/RPA3/PMA0/RA3
- new net N$22: IC1.SOSCI/RPB4/RB4, R22.1
- new net N$24: LED1.A, R22.2
- net +3V3: now also R21.2; no longer JP1.2
- net GND: now also C20.2, LED1.C
- net N$1: now also IC1.PGEC1/AN3/C1INC/C2INA/RPB1/CTED12/PMD1/RB1; no longer IC1.OSC2/CLKO/RPA3/PMA0/RA3
- net N$20: now also R21.1
- net N$4: now also IC1.AN5/C1INA/C2INC/RTCC/RPB3/SCL2/PMWR/RB3; no longer IC1.SOSCI/RPB4/RB4
- net REPORT_N: no longer AVALON1.REPORT_P, R3.1
- net REPORT_P: now also AVALON1.REPORT_P, R3.1
Other:
- moved on the sheet: JP1, R19, U1RX, U1TX
